File: Production/breakouts.kicad_sch (KiCad schematic)
At the start: 1 part, among them J6 Program

Commit message: Pretty solid I redesign
Rotated mcu and reassigned pins for better layout, swapped ldo
Parts:
- removed J6: Program, Connector_PinSocket_2.54mm:PinSocket_1x04_P2.54mm_Vertical, symbol Connector:Conn_01x04_Socket
