File: Production/untitled.kicad_sch (KiCad schematic)
At the start: 7 parts, among them J13 FH34SRJ-16S-0.5SH_50_

Commit message: Tweaked some cap sizes & layout accordingly
Parts:
- C10, C11, C12, C9: footprint Capacitor_SMD:C_0402_1005Metric -> Capacitor_SMD:C_0603_1608Metric
Changed lines of the file:
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@@
 			)
 		)
-		(property "Footprint" "Capacitor_SMD:C_0402_1005Metric"
+		(property "Footprint" "Capacitor_SMD:C_0603_1608Metric"
 			(at 87.63 49.8348 0)
 			(effects
@@
 			)
 		)
-		(property "Footprint" "Capacitor_SMD:C_0402_1005Metric"
+		(property "Footprint" "Capacitor_SMD:C_0603_1608Metric"
 			(at 87.9348 82.55 0)
 			(effects
@@
 			)
 		)
-		(property "Footprint" "Capacitor_SMD:C_0402_1005Metric"
+		(property "Footprint" "Capacitor_SMD:C_0603_1608Metric"
 			(at 101.9048 91.44 0)
 			(effects
@@
 			)
 		)
-		(property "Footprint" "Capacitor_SMD:C_0402_1005Metric"
+		(property "Footprint" "Capacitor_SMD:C_0603_1608Metric"
 			(at 90.17 55.5752 0)
 			(effects

Commit message: Updated BOM to include part numbers
Parts:
- C10, C12: Part Number (none) -> CL10B105KP8NNNC; URL (none) -> https://www.digikey.com/en/products/detail/samsung-electro-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
- C11, C9: Part Number (none) -> CL10A106KQ8NNNL; URL (none) -> https://www.digikey.com/en/products/detail/samsung-electro-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
- J13: Part Number (none) -> FH34SRJ-16S-0.5SH(50); URL (none) -> https://www.digikey.com/en/products/detail/hirose-electric-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
- R6: Part Number (none) -> ESR03EZPJ512; URL (none) -> https://www.digikey.com/en/products/detail/rohm-semiconduct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
- R7: Part Number (none) -> RC0603JR-07680KL; URL (none) -> https://www.digikey.com/en/products/detail/yageo/RC0603JR-0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
Changed lines of the file:
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@@
+			)
+		)
+		(property "Part Number" "RC0603JR-07680KL"
+			(at 95.25 58.42 0)
+			(effects
+				(font
+					(size 1.27 1.27)
+				)
+				(hide yes)
+			)
+		)
+		(property "URL" "https://www.digikey.com/en/products/detail/yageo/RC0603JR-07680KL/726820"
+			(at 95.25 58.42 0)
+			(effects
+				(font
+					(size 1.27 1.27)
+				)
+				(hide yes)
 			)
 		)
@@
 			)
 		)
+		(property "Part Number" "FH34SRJ-16S-0.5SH(50)"
+			(at 118.11 71.12 0)
+			(effects
+				(font
+					(size 1.27 1.27)
+				)
+				(hide yes)
+			)
+		)
+		(property "URL" "https://www.digikey.com/en/products/detail/hirose-electric-co-ltd/FH34SRJ-16S-0-5SH-50/5132522"
+			(at 118.11 71.12 0)
+			(effects
+				(font
+					(size 1.27 1.27)
+				)
+				(hide yes)
+			)
+		)
 		(pin "14"
 		)
@@
 			)
 		)
+		(property "Part Number" "ESR03EZPJ512"
+			(at 91.44 68.58 0)
+			(effects
+				(font
+					(size 1.27 1.27)
+				)
+				(hide yes)
+			)
+		)
+		(property "URL" "https://www.digikey.com/en/products/detail/rohm-semiconductor/ESR03EZPJ512/1762735"
+			(at 91.44 68.58 0)
+			(effects
+				(font
+					(size 1.27 1.27)
+				)
+				(hide yes)
+			)
+		)
 		(pin "1"
 		)
@@
 		)
 		(property "Description" "Unpolarized capacitor"
+			(at 83.82 50.8 0)
+			(effects
+				(font
+					(size 1.27 1.27)
+				)
+				(hide yes)
+			)
+		)
+		(property "Part Number" "CL10A106KQ8NNNL"
+			(at 83.82 50.8 0)
+			(effects
+				(font
+					(size 1.27 1.27)
+				)
+				(hide yes)
+			)
+		)
+		(property "URL" "https://www.digikey.com/en/products/detail/samsung-electro-mechanics/CL10A106KQ8NNNL/3894251"
 			(at 83.82 50.8 0)
 			(effects
@@
 			)
 		)
+		(property "Part Number" "CL10B105KP8NNNC"
+			(at 88.9 86.36 0)
+			(effects
+				(font
+					(size 1.27 1.27)
+				)
+				(hide yes)
+			)
+		)
+		(property "URL" "https://www.digikey.com/en/products/detail/samsung-electro-mechanics/CL10B105KP8NNNC/3887604"
+			(at 88.9 86.36 0)
+			(effects
+				(font
+					(size 1.27 1.27)
+				)
+				(hide yes)
+			)
+		)
 		(pin "1"
 		)
@@
 			)
 		)
+		(property "Part Number" "CL10B105KP8NNNC"
+			(at 102.87 95.25 0)
+			(effects
+				(font
+					(size 1.27 1.27)
+				)
+				(hide yes)
+			)
+		)
+		(property "URL" "https://www.digikey.com/en/products/detail/samsung-electro-mechanics/CL10B105KP8NNNC/3887604"
+			(at 102.87 95.25 0)
+			(effects
+				(font
+					(size 1.27 1.27)
+				)
+				(hide yes)
+			)
+		)
 		(pin "1"
 		)
@@
 			(at 93.98 54.61 0)
 			(effects
+				(font
+					(size 1.27 1.27)
+				)
+				(hide yes)
+			)
+		)
+		(property "Part Number" "CL10A106KQ8NNNL"
+			(at 93.98 54.61 0)
+			(effects
+				(font
+					(size 1.27 1.27)
+				)
+				(hide yes)
+			)
+		)
+		(property "URL" "https://www.digikey.com/en/products/detail/samsung-electro-mechanics/CL10A106KQ8NNNL/3894251"
+			(at 93.98 54.61 0)
+			(effects
