File: Production/Production.kicad_sch (KiCad schematic)
At the start: 28 parts, among them IC1 MAX3323EEPE+, IC2 AP7375-33SA-7, J1 530480510, J2 530480410, J3 USB4085-GF-A_REVB, U2 ADR02AUJZ-REEL7, U3 ATSAMD21G18A-AUT, Y1 32.768, 12.5pF

Commit message: more of previous
Parts:
- S1, S2: footprint FSM4JH -> FSM10JH:FSM4JH
Changed lines of the file:
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@@
 			)
 		)
-		(property "Footprint" "FSM4JH"
+		(property "Footprint" "FSM10JH:FSM4JH"
 			(at 63.5 221.92 0)
 			(effects
@@
 			)
 		)
-		(property "Footprint" "FSM4JH"
+		(property "Footprint" "FSM10JH:FSM4JH"
 			(at 63.5 237.16 0)
 			(effects
