File: Production v1.1/untitled.kicad_sch (KiCad schematic)
At the start: 7 parts, among them J13 FH34SRJ-16S-0.5SH_50_

Commit message: Better v1.1, but I can do better
Parts:
- R6, R7: footprint Resistor_SMD:R_0603_1608Metric -> Resistor_SMD:R_0201_0603Metric
Changed lines of the file:
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@@
 			)
 		)
-		(property "Footprint" "Resistor_SMD:R_0603_1608Metric"
+		(property "Footprint" "Resistor_SMD:R_0201_0603Metric"
 			(at 95.25 60.198 90)
 			(effects
@@
 		)
 		(instances
-			(project "Production v2"
+			(project "Production v1.1"
 				(path "/36880c03-5560-4777-bc12-f18c70ba2db4/7bd35dc1-a7c7-48b2-b6a6-7456ace66990"
 					(reference "R7")
@@
 		)
 		(instances
-			(project "Production v2"
+			(project "Production v1.1"
 				(path "/36880c03-5560-4777-bc12-f18c70ba2db4/7bd35dc1-a7c7-48b2-b6a6-7456ace66990"
 					(reference "#PWR037")
@@
 		)
 		(instances
-			(project "Production v2"
+			(project "Production v1.1"
 				(path "/36880c03-5560-4777-bc12-f18c70ba2db4/7bd35dc1-a7c7-48b2-b6a6-7456ace66990"
 					(reference "#PWR036")
@@
 		)
 		(instances
-			(project "Production v2"
+			(project "Production v1.1"
 				(path "/36880c03-5560-4777-bc12-f18c70ba2db4/7bd35dc1-a7c7-48b2-b6a6-7456ace66990"
 					(reference "#PWR038")
@@
 		)
 		(instances
-			(project "Production v2"
+			(project "Production v1.1"
 				(path "/36880c03-5560-4777-bc12-f18c70ba2db4/7bd35dc1-a7c7-48b2-b6a6-7456ace66990"
 					(reference "J13")
@@
 			)
 		)
-		(property "Footprint" "Resistor_SMD:R_0603_1608Metric"
+		(property "Footprint" "Resistor_SMD:R_0201_0603Metric"
 			(at 91.44 70.358 90)
 			(effects
@@
 		)
 		(instances
-			(project "Production v2"
+			(project "Production v1.1"
 				(path "/36880c03-5560-4777-bc12-f18c70ba2db4/7bd35dc1-a7c7-48b2-b6a6-7456ace66990"
 					(reference "R6")
@@
 		)
 		(instances
-			(project "Production v2"
+			(project "Production v1.1"
 				(path "/36880c03-5560-4777-bc12-f18c70ba2db4/7bd35dc1-a7c7-48b2-b6a6-7456ace66990"
 					(reference "C9")
@@
 		)
 		(instances
-			(project "Production v2"
+			(project "Production v1.1"
 				(path "/36880c03-5560-4777-bc12-f18c70ba2db4/7bd35dc1-a7c7-48b2-b6a6-7456ace66990"
 					(reference "#PWR035")
@@
 		)
 		(instances
-			(project "Production v2"
+			(project "Production v1.1"
 				(path "/36880c03-5560-4777-bc12-f18c70ba2db4/7bd35dc1-a7c7-48b2-b6a6-7456ace66990"
 					(reference "C10")
@@
 		)
 		(instances
-			(project "Production v2"
+			(project "Production v1.1"
 				(path "/36880c03-5560-4777-bc12-f18c70ba2db4/7bd35dc1-a7c7-48b2-b6a6-7456ace66990"
 					(reference "#PWR034")
@@
 		)
 		(instances
-			(project "Production v2"
+			(project "Production v1.1"
 				(path "/36880c03-5560-4777-bc12-f18c70ba2db4/7bd35dc1-a7c7-48b2-b6a6-7456ace66990"
 					(reference "C12")
@@
 		)
 		(instances
-			(project "Production v2"
+			(project "Production v1.1"
 				(path "/36880c03-5560-4777-bc12-f18c70ba2db4/7bd35dc1-a7c7-48b2-b6a6-7456ace66990"
 					(reference "C11")

Commit message: Components are all moved to the bottom layer, top is ground
Parts:
- R6, R7: footprint Resistor_SMD:R_0201_0603Metric -> Resistor_SMD:R_0603_1608Metric
Changed lines of the file:
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@@
 			)
 		)
-		(property "Footprint" "Resistor_SMD:R_0201_0603Metric"
+		(property "Footprint" "Resistor_SMD:R_0603_1608Metric"
 			(at 95.25 60.198 90)
 			(effects
@@
 			)
 		)
-		(property "Footprint" "Resistor_SMD:R_0201_0603Metric"
+		(property "Footprint" "Resistor_SMD:R_0603_1608Metric"
 			(at 91.44 70.358 90)
 			(effects

Commit message: v1.1 sent for assembly
Parts:
- R6, R7: footprint Resistor_SMD:R_0603_1608Metric -> Resistor_SMD:R_0201_0603Metric
Changed lines of the file:
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@@
 			)
 		)
-		(property "Footprint" "Resistor_SMD:R_0603_1608Metric"
+		(property "Footprint" "Resistor_SMD:R_0201_0603Metric"
 			(at 95.25 60.198 90)
 			(effects
@@
 			)
 		)
-		(property "Footprint" "Resistor_SMD:R_0603_1608Metric"
+		(property "Footprint" "Resistor_SMD:R_0201_0603Metric"
 			(at 91.44 70.358 90)
 			(effects

Commit message: Updated v1.1 and re-ordered
One net was not connected
Parts:
- J13: MANUFACTURER HRS -> (none)
- R6: Part Number ESR03EZPJ512 -> ERJ-1GNF5101C; URL https://www.digikey.com/en/products/detail/rohm-semiconduct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 -> https://www.digikey.com/en/products/detail/panasonic-electr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
- R7: Part Number RC0603JR-07680KL -> ERJ-1GNF6803C; URL https://www.digikey.com/en/products/detail/yageo/RC0603JR-0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 -> https://www.digikey.com/en/products/detail/panasonic-electr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
Changed lines of the file:
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@@
 			)
 		)
-		(property "Part Number" "RC0603JR-07680KL"
+		(property "Part Number" "ERJ-1GNF6803C"
 			(at 95.25 58.42 0)
 			(effects
@@
 			)
 		)
-		(property "URL" "https://www.digikey.com/en/products/detail/yageo/RC0603JR-07680KL/726820"
+		(property "URL" "https://www.digikey.com/en/products/detail/panasonic-electronic-components/ERJ-1GNF6803C/2036436"
 			(at 95.25 58.42 0)
 			(effects
@@
 			)
 		)
-		(property "MANUFACTURER" "HRS"
-			(at 118.11 71.12 0)
-			(effects
-				(font
-					(size 1.27 1.27)
-				)
-				(justify bottom)
-				(hide yes)
-			)
-		)
 		(property "Part Number" "FH34SRJ-16S-0.5SH(50)"
 			(at 118.11 71.12 0)
@@
 			)
 		)
-		(property "Part Number" "ESR03EZPJ512"
+		(property "Part Number" "ERJ-1GNF5101C"
 			(at 91.44 68.58 0)
 			(effects
@@
 			)
 		)
-		(property "URL" "https://www.digikey.com/en/products/detail/rohm-semiconductor/ESR03EZPJ512/1762735"
+		(property "URL" "https://www.digikey.com/en/products/detail/panasonic-electronic-components/ERJ-1GNF5101C/2036192"
 			(at 91.44 68.58 0)
 			(effects
