File: Production v1.2/untitled.kicad_sch (KiCad schematic)
At the start: 7 parts, among them J4 FH34SRJ-16S-0.5SH_50_

Commit message: v1.2 checked & labeled
flipped fpc connector to underside, for better ribbon routing.
Connections:
- net +3V3: now also J4.5, J4.7; no longer J4.10, J4.12
- net GND: now also J4.16, J4.6; no longer J4.1, J4.11
- net MOSI: now also J4.12; no longer J4.5
- net OLED_CS: now also J4.8; no longer J4.9
- net OLED_DC: now also J4.10; no longer J4.7
- net OLED_RST: now also J4.9; no longer J4.8
- net SCK: now also J4.11; no longer J4.6
- net at R8.2: now also J4.13; no longer J4.4
- net at C10.2: now also J4.4; no longer J4.13
- net at C10.1: now also J4.3; no longer J4.14
- net at J4.15: now also C9.2; no longer C12.2
- net at C12.1: now also J4.1; no longer J4.16
- net at J4.2: now also C12.2; no longer C9.2
- net at C11.1: now also J4.14; no longer J4.3
Changed lines of the file:
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@@
 		(dnp no)
 		(fields_autoplaced yes)
-		(property "Reference" "#PWR027"
+		(property "Reference" "#PWR025"
 			(at 107.95 45.72 0)
 			(effects
@@
 			(project "Production v1.2"
 				(path "/36880c03-5560-4777-bc12-f18c70ba2db4/7bd35dc1-a7c7-48b2-b6a6-7456ace66990"
-					(reference "#PWR027")
+					(reference "#PWR025")
 					(unit 1)
 				)
@@
 		(on_board yes)
 		(dnp no)
-		(property "Reference" "#PWR026"
+		(property "Reference" "#PWR024"
 			(at 100.33 81.28 0)
 			(effects
@@
 			(project "Production v1.2"
 				(path "/36880c03-5560-4777-bc12-f18c70ba2db4/7bd35dc1-a7c7-48b2-b6a6-7456ace66990"
-					(reference "#PWR026")
+					(reference "#PWR024")
 					(unit 1)
 				)
@@
 		(dnp no)
 		(fields_autoplaced yes)
-		(property "Reference" "#PWR028"
+		(property "Reference" "#PWR026"
 			(at 130.81 105.41 0)
 			(effects
@@
 			(project "Production v1.2"
 				(path "/36880c03-5560-4777-bc12-f18c70ba2db4/7bd35dc1-a7c7-48b2-b6a6-7456ace66990"
-					(reference "#PWR028")
-					(unit 1)
-				)
-			)
-		)
-	)
-	(symbol
-		(lib_id "FH34SRJ-16S-0.5SH_50_:FH34SRJ-16S-0.5SH_50_")
-		(at 118.11 71.12 0)
-		(unit 1)
-		(exclude_from_sim no)
-		(in_bom yes)
-		(on_board yes)
-		(dnp no)
-		(property "Reference" "J4"
-			(at 126.746 49.784 0)
-			(effects
-				(font
-					(size 1.27 1.27)
-				)
-			)
-		)
-		(property "Value" "FH34SRJ-16S-0.5SH_50_"
-			(at 137.414 52.578 0)
-			(effects
-				(font
-					(size 1.27 1.27)
-				)
-			)
-		)
-		(property "Footprint" "FH34SRJ_16S_0_5SH_50:HRS_FH34SRJ-16S-0.5SH_50_"
-			(at 118.11 71.12 0)
-			(effects
-				(font
-					(size 1.27 1.27)
-				)
-				(justify bottom)
-				(hide yes)
-			)
-		)
-		(property "Datasheet" ""
-			(at 118.11 71.12 0)
-			(effects
-				(font
-					(size 1.27 1.27)
-				)
-				(hide yes)
-			)
-		)
-		(property "Description" ""
-			(at 118.11 71.12 0)
-			(effects
-				(font
-					(size 1.27 1.27)
-				)
-				(hide yes)
-			)
-		)
-		(property "Part Number" "FH34SRJ-16S-0.5SH(50)"
-			(at 118.11 71.12 0)
-			(effects
-				(font
-					(size 1.27 1.27)
-				)
-				(hide yes)
-			)
-		)
-		(property "URL" "https://www.digikey.com/en/products/detail/hirose-electric-co-ltd/FH34SRJ-16S-0-5SH-50/5132522"
-			(at 118.11 71.12 0)
-			(effects
-				(font
-					(size 1.27 1.27)
-				)
-				(hide yes)
-			)
-		)
-		(pin "14"
-		)
-		(pin "15"
-		)
-		(pin "16"
-		)
-		(pin "2"
-		)
-		(pin "3"
-		)
-		(pin "4"
-		)
-		(pin "10"
-		)
-		(pin "1"
-		)
-		(pin "5"
-		)
-		(pin "6"
-		)
-		(pin "7"
-		)
-		(pin "8"
-		)
-		(pin "12"
-		)
-		(pin "9"
-		)
-		(pin "S1"
-		)
-		(pin "S2"
-		)
-		(pin "13"
-		)
-		(pin "11"
-		)
-		(instances
-			(project "Production v1.2"
-				(path "/36880c03-5560-4777-bc12-f18c70ba2db4/7bd35dc1-a7c7-48b2-b6a6-7456ace66990"
-					(reference "J4")
+					(reference "#PWR026")
 					(unit 1)
 				)
@@
 		(dnp no)
 		(fields_autoplaced yes)
-		(property "Reference" "#PWR025"
+		(property "Reference" "#PWR023"
 			(at 82.55 67.31 0)
 			(effects
@@
 			(project "Production v1.2"
 				(path "/36880c03-5560-4777-bc12-f18c70ba2db4/7bd35dc1-a7c7-48b2-b6a6-7456ace66990"
-					(reference "#PWR025")
+					(reference "#PWR023")
 					(unit 1)
 				)
@@
 		(dnp no)
 		(fields_autoplaced yes)
-		(property "Reference" "#PWR024"
+		(property "Reference" "#PWR022"
 			(at 74.93 74.93 0)
 			(effects
@@
 			(project "Production v1.2"
 				(path "/36880c03-5560-4777-bc12-f18c70ba2db4/7bd35dc1-a7c7-48b2-b6a6-7456ace66990"
-					(reference "#PWR024")
+					(reference "#PWR022")
 					(unit 1)
 				)
@@
 					(unit 1)
 				)
+			)
+		)
+	)
+	(symbol
+		(lib_name "FH34SRJ-16S-0.5SH_50__1")
+		(lib_id "FH34SRJ-16S-0.5SH_50_:FH34SRJ-16S-0.5SH_50_")
+		(at 118.11 71.12 0)
+		(unit 1)
+		(exclude_from_sim no)
+		(in_bom yes)
+		(on_board yes)
+		(dnp no)
+		(property "Reference" "J4"
+			(at 126.746 49.784 0)
+			(effects
+				(font
+					(size 1.27 1.27)
+				)
+			)
+		)
+		(property "Value" "FH34SRJ-16S-0.5SH_50_"
+			(at 137.414 52.578 0)
+			(effects
+				(font
+					(size 1.27 1.27)
+				)
+			)
+		)
+		(property "Footprint" "FH34SRJ_16S_0_5SH_50:HRS_FH34SRJ-16S-0.5SH_50_"
+			(at 118.11 71.12 0)
+			(effects
+				(font
+					(size 1.27 1.27)
+				)
+				(justify bottom)
+				(hide yes)
+			)
+		)
+		(property "Datasheet" ""
+			(at 118.11 71.12 0)
+			(effects
+				(font
+					(size 1.27 1.27)
+				)
+				(hide yes)
+			)
+		)
+		(property "Description" ""
+			(at 118.11 71.12 0)
+			(effects
+				(font
+					(size 1.27 1.27)
+				)
+				(hide yes)
+			)
+		)
+		(property "Part Number" "FH34SRJ-16S-0.5SH(50)"
+			(at 118.11 71.12 0)
+			(effects
+				(font
+					(size 1.27 1.27)
+				)
+				(hide yes)
+			)
+		)
+		(property "URL" "https://www.digikey.com/en/products/detail/hirose-electric-co-ltd/FH34SRJ-16S-0-5SH-50/5132522"
+			(at 118.11 71.12 0)
+			(effects
+				(font
+					(size 1.27 1.27)
+				)
+				(hide yes)
+			)
+		)
+		(pin "14"
+		)
+		(pin "15"
+		)
+		(pin "16"
+		)
+		(pin "2"
+		)
+		(pin "3"
+		)
+		(pin "4"
+		)
+		(pin "10"
+		)
+		(pin "1"
+		)
+		(pin "5"
+		)
+		(pin "6"
+		)
+		(pin "7"
+		)
+		(pin "8"
+		)
+		(pin "12"
+		)
+		(pin "9"
+		)
+		(pin "S1"
+		)
+		(pin "S2"
+		)
+		(pin "13"
+		)
+		(pin "11"
+		)
+		(instances
+			(project "Production v1.2"
+				(path "/36880c03-5560-4777-bc12-f18c70ba2db4/7bd35dc1-a7c7-48b2-b6a6-7456ace66990"
+					(reference "J4")
+					(unit 1)
+				)
